File: MCU Datalogger.kicad_sch (KiCad schematic)
At the start: 25 parts, among them U1 24LC1025, U2 24LC1025, U3 DS1337S_, U4 ATMEGA328P-AU, Y1 16 MHz, Y2 32.768kHz

Commit message: abc123 label fixed
Connections:
- net AREF: no longer D2.1 (K), R2.2
- new net abc123: D2.1 (K), R2.2
Changed lines of the file:
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@@
     (rev "1")
   )
-  (junction (at 168.766 52.1795) (diameter 0) (color 0 0 0 0)
-  )
   (junction (at 104.6347 128.4498) (diameter 0) (color 0 0 0 0)
   )
@@
   )
   (junction (at 154.4415 73.4438) (diameter 0) (color 0 0 0 0)
-  )
-  (junction (at 171.2592 40.1239) (diameter 0) (color 0 0 0 0)
   )
   (junction (at 253.2251 42.666) (diameter 0) (color 0 0 0 0)
@@
     (stroke (width 0) (type default))
   )
-  (wire (pts (xy 168.766 52.1795) (xy 168.766 40.1239))
-    (stroke (width 0) (type default))
-  )
   (wire (pts (xy 165.3774 142.7882) (xy 168.4831 142.7882))
     (stroke (width 0) (type default))
@@
     (stroke (width 0) (type default))
   )
-  (wire (pts (xy 168.766 40.1239) (xy 171.2592 40.1239))
-    (stroke (width 0) (type default))
-  )
   (wire (pts (xy 240.7316 70.0072) (xy 240.8066 70.0072))
     (stroke (width 0) (type default))
@@
     (stroke (width 0) (type default))
   )
-  (wire (pts (xy 168.766 52.1795) (xy 178.1691 52.1795))
-    (stroke (width 0) (type default))
-  )
   (wire (pts (xy 168.4831 131.4211) (xy 168.4831 131.6708))
     (stroke (width 0) (type default))
@@
     (stroke (width 0) (type default))
   )
-  (wire (pts (xy 164.2876 52.1795) (xy 168.766 52.1795))
+  (wire (pts (xy 164.2876 52.1795) (xy 178.1691 52.1795))
     (stroke (width 0) (type default))
   )
@@
     (effects (font (size 1.27 1.27)) (justify left bottom))
   )
+  (label "abc123" (at 167.2611 52.1795 0) (fields_autoplaced)
+    (effects (font (size 1.27 1.27)) (justify left bottom))
+  )
   (label "Vcc" (at 30.7714 135.6874 0) (fields_autoplaced)
     (effects (font (size 1.27 1.27)) (justify left bottom))
@@
     (effects (font (size 1.27 1.27)) (justify right bottom))
   )
-  (label "abc123" (at 168.766 52.1795 0) (fields_autoplaced)
-    (effects (font (size 1.27 1.27)) (justify left bottom))
-  )
   (label "D4" (at 230.1347 60.446 0) (fields_autoplaced)
